File: ESP 32 Low Power.kicad_pcb (KiCad board)
At the start: 2 copper layers, 100 x 50 mm, 37 parts, among them J1 Conn_01x02, J2 Conn_01x02, J3 Conn_01x18, J4 Conn_01x18, J5 Conn_01x02, P1 USB_C, Q1 DMG2301L, Q2 S8050, Q3 S8050, U1 XC6220B331MR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

Commit message: Added battery low voltage protection
Parts:
- added C7: 0.1uF, Capacitor_SMD:C_0805_2012Metric_Pad1.15x1.40mm_HandSolder, F.Cu at (141.4, 88.0)
- added Q4: SE8810A, Package_TO_SOT_SMD:SOT-23-6_Handsoldering, F.Cu at (140.0, 99.3)
- added R10: 100R, Resistor_SMD:R_0805_2012Metric_Pad1.15x1.40mm_HandSolder, F.Cu at (143.5, 88.0)
- added R11: 1K, Resistor_SMD:R_0805_2012Metric_Pad1.15x1.40mm_HandSolder, F.Cu at (143.3, 94.4)
- added U5: DW01B, Package_TO_SOT_SMD:SOT-23-6_Handsoldering, F.Cu at (140.0, 93.4)
- J5: value Conn_01x02 -> Battery
- U2: value CN3063 -> PMIC-CN3063(SOIC8)
- moved J5 3.47 mm to (138.7, 88.8), turned to 180 degrees
Connections:
- J5 pad 1: +BATT -> Net-(C7-Pad2)
- J5 pad 2: GND -> +BATT
Routing:
- net +3V3: track 104.4 -> 134.3 mm
- net /CHIP_PU: track 80.5 -> 98.5 mm
- net Net-(C7-Pad2): track 0.00 -> 17.5 mm
- net Net-(C7-Pad1): track 0.00 -> 5.77 mm
- net GND: track 120.6 -> 126.0 mm, vias 46 -> 48
- net Net-(R11-Pad1): track 0.00 -> 4.34 mm
- net +BATT: track 42.2 -> 45.9 mm
- net Net-(Q4-Pad6): track 0.00 -> 3.19 mm
- net Net-(Q4-Pad4): track 0.00 -> 3.19 mm
- net Net-(Q4-Pad2): track 0.00 -> 2.70 mm

Commit message: Some better placement
Parts:
- U2: value PMIC-CN3063(SOIC8) -> CN3063
- moved R11 19.4 mm to (124.2, 90.9)
- moved U5 12.0 mm to (128.2, 90.9), turned to 180 degrees
- moved Q4 10.2 mm to (134.1, 90.9), turned to 180 degrees
- moved Q2 0.89 mm to (129.7, 97.0)
Routing:
- net +3V3: track 134.3 -> 112.2 mm
- net Net-(C7-Pad1): track 5.77 -> 23.1 mm
- net /CHIP_PU: track 98.5 -> 84.3 mm
- net Net-(R11-Pad1): track 4.34 -> 7.80 mm
- net +BATT: track 45.9 -> 48.8 mm
- net GND: track 126.0 -> 123.2 mm
- net Net-(C7-Pad2): track 17.5 -> 19.8 mm
